File: ESSync.kicad_sch (KiCad schematic)
At the start: 9 parts, among them SW1 SW_Slide_DPDT, U3 ESP32-C3-DevKitM-1

Commit message: Added updated files of pcb
Parts:
- removed MT3608, TP4056: Conn_01x04, Connector:FanPinHeader_1x04_P2.54mm_Vertical, symbol Connector_Generic:Conn_01x04
- added J1, J2: Conn_01x15, Connector_PinSocket_2.54mm:PinSocket_1x15_P2.54mm_Vertical, symbol Connector_Generic:Conn_01x15
- added J10, J11, J12, J5, J6, J7, J8, J9: Conn_01x01, Connector_PinHeader_1.00mm:PinHeader_1x01_P1.00mm_Vertical, symbol Connector_Generic:Conn_01x01
- added J3, J4: Conn_01x15, Connector_PinHeader_2.54mm:PinHeader_1x15_P2.54mm_Vertical, symbol Connector_Generic:Conn_01x15
- SPI_SCREEN1: footprint Connector_PinHeader_2.54mm:PinHeader_1x07_P2.54mm_Vertical -> Connector_PinSocket_2.54mm:PinSocket_1x07_P2.54mm_Vertical
Connections:
- net +3.3V: now also J2.2 (3V3)
- net +5V: now also J9.1 (Pin_1)
- net BAT+: now also J11.1 (Pin_1)
- net BAT-: now also J12.1 (Pin_1)
- net DC: now also J2.5 (GPIO3); no longer U3.5 (IO3)
- net GND: now also J1.1 (GND), J10.1 (Pin_1)
- net IN+: now also J7.1 (Pin_1)
- net IN-: now also J6.1 (Pin_1), J8.1 (Pin_1)
- net OUT+: now also J5.1 (Pin_1)
- net RES: now also J1.11 (GPIO4); no longer U3.20 (IO4)
- net SCL_SPI: now also J1.8 (GPIO7); no longer U3.23 (IO7)
- net SDA_SPI: now also J1.9 (GPIO6); no longer U3.22 (IO6)
Other:
- note added: "1"
- note added: "23/06/2026"
- note added: "BOTTOM PCB"
- note added: "ESP 32 C3"
- note added: "ESP 32 C3 Connector Female Pins"
- note added: "ESP 32 C3 Connector Pins Male"
- note added: "ESP 32 PON/OFF SWITCH"
- note added: "ESSYNC SCHEMATIC"
- note added: "GLOBAL POWER SWITCH"
- note added: "MT3608"
- note added: "SPI Screen Connector Male Pins"
- note added: "TP4056"
- note added: "Top PCB"
- moved on the sheet: Battery1, C1, MPU6050, S1, SPI_SCREEN1, SW1, U3
