File: src/PCB/ESS_Top/ESS_Top.kicad_pcb (KiCad board)
At the start: 2 copper layers, 45.7 x 39.9 mm, 3 parts, among them J1 Conn_01x15, J2 Conn_01x15

Commit message: added ground fill
Routing:
- added copper zone on B.Cu, net GND
Changed lines of the file:
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@@
 		(net 23)
+	)
+	(zone
+		(net 13)
+		(net_name "GND")
+		(layer "B.Cu")
+		(hatch edge 0.5)
+		(connect_pads
+			(clearance 0.5)
+		)
+		(min_thickness 0.25)
+		(filled_areas_thickness no)
+		(fill yes
+			(thermal_gap 0.5)
+			(thermal_bridge_width 0.5)
+		)
+		(polygon
+			(pts
+				(xy 124.82 81.01) (xy 124.35 119.95) (xy 168.67 120.21) (xy 168.67 80.8) (xy 124.81 81.07)
+			)
+		)
 	)
 	(embedded_fonts no)
